File: hardware/MP3 Shield.sch (EAGLE design)
At the start: 71 parts, among them Q1 12.288MHz, U1 3.3V, U2 ARDUINO_R3_SHIELD, U3 VS1053, U4 1.8V, U6 USD-SOCKET, U7 74HC4050 LVL CONVERTER

Commit message: Final touches to layout
Connections:
- net 3.3V: no longer R5.1
- net GND: now also R5.1
Other:
- note added: "RST now pulled low by default"
- moved on the sheet: R5

Commit message: Adding transistor part #s
Commits at 32,000 ft! Whooo!
Parts:
- Q2, Q3: value (none) -> PMBT3906
- Q4, Q5: value (none) -> MMBT2222
Changed lines of the file:
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@@
 <part name="C19" library="SparkFun" deviceset="CAP" device="0603-CAP" value="3.3nF"/>
 <part name="C20" library="SparkFun" deviceset="CAP" device="0603-CAP" value="3.3nF"/>
-<part name="Q2" library="SparkFun-DiscreteSemi" deviceset="TRANSISTOR_PNP" device="SMD"/>
-<part name="Q3" library="SparkFun-DiscreteSemi" deviceset="TRANSISTOR_PNP" device="SMD"/>
-<part name="Q4" library="SparkFun-DiscreteSemi" deviceset="TRANSISTOR_NPN" device="SOT23-3"/>
-<part name="Q5" library="SparkFun-DiscreteSemi" deviceset="TRANSISTOR_NPN" device="SOT23-3"/>
+<part name="Q2" library="SparkFun-DiscreteSemi" deviceset="TRANSISTOR_PNP" device="SMD" value="PMBT3906"/>
+<part name="Q3" library="SparkFun-DiscreteSemi" deviceset="TRANSISTOR_PNP" device="SMD" value="PMBT3906"/>
+<part name="Q4" library="SparkFun-DiscreteSemi" deviceset="TRANSISTOR_NPN" device="SOT23-3" value="MMBT2222"/>
+<part name="Q5" library="SparkFun-DiscreteSemi" deviceset="TRANSISTOR_NPN" device="SOT23-3" value="MMBT2222"/>
 <part name="GND29" library="SparkFun" deviceset="GND" device=""/>
 <part name="GND30" library="SparkFun" deviceset="GND" device=""/>
@@
 <instance part="C19" gate="G$1" x="281.94" y="66.04"/>
 <instance part="C20" gate="G$1" x="281.94" y="33.02"/>
-<instance part="Q2" gate="G$1" x="335.28" y="40.64" rot="MR0"/>
-<instance part="Q3" gate="G$1" x="335.28" y="73.66" rot="MR0"/>
-<instance part="Q4" gate="G$1" x="314.96" y="33.02" rot="MR0"/>
-<instance part="Q5" gate="G$1" x="314.96" y="66.04" rot="MR0"/>
+<instance part="Q2" gate="G$1" x="335.28" y="40.64" smashed="yes" rot="MR0">
+<attribute name="NAME" x="337.82" y="38.1" size="1.778" layer="95" rot="MR180"/>
+<attribute name="VALUE" x="335.28" y="35.56" size="1.778" layer="96" rot="MR180"/>
+</instance>
+<instance part="Q3" gate="G$1" x="335.28" y="73.66" smashed="yes" rot="MR0">
+<attribute name="NAME" x="337.82" y="71.12" size="1.778" layer="95" rot="MR180"/>
+<attribute name="VALUE" x="335.28" y="68.58" size="1.778" layer="96" rot="MR180"/>
+</instance>
+<instance part="Q4" gate="G$1" x="314.96" y="33.02" smashed="yes" rot="MR0">
+<attribute name="NAME" x="317.5" y="30.48" size="1.778" layer="95" rot="MR180"/>
+<attribute name="VALUE" x="314.96" y="27.94" size="1.778" layer="96" rot="MR180"/>
+</instance>
+<instance part="Q5" gate="G$1" x="314.96" y="66.04" smashed="yes" rot="MR0">
+<attribute name="NAME" x="317.5" y="63.5" size="1.778" layer="95" rot="MR180"/>
+<attribute name="VALUE" x="314.96" y="60.96" size="1.778" layer="96" rot="MR180"/>
+</instance>
 <instance part="GND29" gate="1" x="312.42" y="22.86"/>
 <instance part="GND30" gate="1" x="281.94" y="58.42"/>

Commit message: Added ISP connector for compatibility with Lenoardo/Mega.
Routed SPI pins to ISP connector for more compatibility between Arduino
versions.
Parts:
- removed FRAME2: FRAME-LETTER, SparkFun-Aesthetics:FRAME-LETTER
- added FRAME1: FRAME-LEDGER, SparkFun-Aesthetics:FRAME-LEDGER
- added J1: ISP/SPI, SparkFun:AVR_SPI_PRG_6PTH
Connections:
- removed net N$13: SJ4.2, U2.*D10
- new net 5V-MUTE: SJ4.2, U2.*D5
- net 5V-MOSI: now also J1.4
- net 5V-SCK: now also J1.3
- net GND: now also J1.6
- net MISO: now also J1.1
- net VCC: now also J1.2
Other:
- note added: "Populate with 2x3 female connector to be compatible with Leonardo/Mega"
- note removed: "Find default NPN and PNP SMD"
- note removed: "Reduce size of SparkFun schematic symbol"
- moved on the sheet: C1, C10, C11, C12, C13, C14, C15, C16, C17, C18, C19, C2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

Commit message: Finished up and removed TODOs
Other:
- note removed: "Push 3.5mm R/L schematic symbol to main fp branch"
- note removed: "Todo"
Changed lines of the file:
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@@
 <text x="327.66" y="269.24" size="1.778" layer="97">Added microSD</text>
 <text x="327.66" y="266.7" size="1.778" layer="97">Added 74HC4050 LVL Converter</text>
-<text x="327.66" y="223.52" size="1.778" layer="97">Push 3.5mm R/L schematic symbol to main fp branch</text>
 <text x="325.12" y="256.54" size="1.778" layer="97">New on v1.4:</text>
-<text x="325.12" y="226.06" size="1.778" layer="97">Todo</text>
 <text x="327.66" y="254" size="1.778" layer="97">Added solder jumper to select between GBUF and GND</text>
 <text x="370.84" y="172.72" size="1.778" layer="97">Connect GBUF if attaching amplifier</text>

Commit message: Updated 3.5mm jack and HEX inverter footprints.
Parts:
- C1, C17, C18, C6: device SparkFun:CAP_POL1206 -> SparkFun-Capacitors:10UF-16V-10%(TANT)
- C10, C11: device SparkFun:CAP0603-CAP -> SparkFun-Capacitors:10NF/10000PF-50V-10%(0603)
- C12: device SparkFun:CAP0603-CAP -> SparkFun-Capacitors:47NF(0.047UF/47000PF)-25V-5%(0603)SMD
- C13, C14, C15, C16, C2, C5, C7: device SparkFun:CAP0603-CAP -> SparkFun-Capacitors:0.1UF-25V(+80/-20%)(0603)
- C19, C20: device SparkFun:CAP0603-CAP -> SparkFun-Capacitors:3.3NF-100V-10%(0603)
- C3, C8: device SparkFun:CAP0603-CAP -> SparkFun-Capacitors:22PF-50V-5%(0603)
- C4: device SparkFun:CAP0603-CAP -> SparkFun-Capacitors:470PF-50V-5%(0603)SMD
- C9: device SparkFun:CAP0603-CAP -> SparkFun-Capacitors:1.0UF-16V-10%(0603)
- JP1: device SparkFun:AUDIO-JACKSMD2 -> SparkFun-Connectors:AUDIO-JACKSMD2
- LED1: device SparkFun:LED0603 -> SparkFun-LED:LED-RED0603
- Q2, Q3: device SparkFun-DiscreteSemi:TRANSISTOR_PNPSMD -> SparkFun-DiscreteSemi:TRANSISTOR_PNPPMBT3906
- Q4, Q5: value MMBT2222 -> MMBT2222A; device SparkFun-DiscreteSemi:TRANSISTOR_NPNSOT23-3 -> SparkFun-DiscreteSemi:TRANSISTOR_NPNMMBT2222A
- R1: device SparkFun:RESISTOR0603-RES -> SparkFun-Resistors:1M-1%
- R10, R11, R12, R2, R24, R3, R4, R5: device SparkFun:RESISTOR0603-RES -> SparkFun-Resistors:100KOHM1/10W1%(0603)
- R13, R14, R23: device SparkFun:RESISTOR0603-RES -> SparkFun-Resistors:1KOHM1/10W1%(0603)
- R15, R16, R17, R18, R19, R20: device SparkFun:RESISTOR0603-RES -> SparkFun-Resistors:10KOHM1/10W1%(0603)0603
- R21, R22: device SparkFun:RESISTOR0603-RES -> SparkFun-Resistors:470OHM1/10W1%(0603)
- R6, R7: device SparkFun:RESISTOR0603-RES -> SparkFun-Resistors:20OHM1/10W1%(0603)SMD
- R8: device SparkFun:RESISTOR0603-RES -> SparkFun-Resistors:330OHM1/10W1%(0603)
- R9: device SparkFun:RESISTOR0603-RES -> SparkFun-Resistors:10OHM1/10W5%0603SMD
- S2: device SparkFun:SWITCH-MOMENTARY-2SMD -> SparkFun-Electromechanical:SWITCH-MOMENTARY-2SMD
- U1: device SparkFun:V_REG_LDOSMD -> SparkFun-PowerIC:V_REG_MIC52053.3V
- U3: device SparkFun:VS1033 -> SparkFun-DigitalIC:VS1033/1053SMD
- U4: device SparkFun:V_REG_LDOSMD2 -> SparkFun-PowerIC:V_REG_SP62141.8V
- U7: device SparkFun:HEX_CONVERTER -> SparkFun-DigitalIC:HEX_CONVERTER
Other:
- note added: "Moved to tighter SOIC FP on HEX inverter"
- note added: "Touched up 3.5mm jack footprint"
